File: BLDC-driver.sch (KiCad schematic (older format))
At the start: 60 parts, among them J1 Conn_01x06, J2 Conn_01x06, Q1 FDMS86550, Q2 FDMS86550, Q3 FDMS86550, Q4 FDMS86550, Q5 FDMS86550, Q6 FDMS86550, U1 ADP3120A, U2 STM32F103C8Tx, U3 AS5600, U4 ADP3120A, U5 ADP3120A, U6 MP2359, U7 MIC5504-3.3YM5

Commit message: Latest
Parts:
- removed U3: AS5600, Package_SO:SOIC-8_3.9x4.9mm_P1.27mm, symbol BLDC-driver-rescue:AS5600
- added C29: 100nF, Capacitor_SMD:C_0603_1608Metric, symbol Device:C_Small
- added C30: 100nF, Capacitor_SMD:C_0402_1005Metric, symbol Device:C_Small
- added D2, D3: LED, LED_SMD:LED_0603_1608Metric, symbol Device:LED
- added D4, D5, D6: 30V, Diode_SMD:D_SOD-523, symbol Device:D_Schottky_Small
- added NT2: Net-Tie_2, NetTie:NetTie-2_SMD_Pad0.5mm, symbol Device:Net-Tie_2
- added R14, R15: 0.001, Resistor_SMD:R_1210_3225Metric, symbol Device:R
- added R16: 120R, Resistor_SMD:R_0603_1608Metric, symbol Device:R_Small
- added R17, R18: 1k, Resistor_SMD:R_0603_1608Metric, symbol Device:R_Small
- added R19, R20: 10k, Resistor_SMD:R_0603_1608Metric, symbol Device:R_Small
- added R21, R22: 10k, Resistor_SMD:R_0402_1005Metric, symbol Device:R_Small
- added U3: MAX3051, Package_TO_SOT_SMD:SOT-23-8, symbol Interface_UART:MAX3051
- added U8, U9: NCS210, Package_TO_SOT_SMD:SOT-363_SC-70-6, symbol Amplifier_Current:NCS210
- C27: value 100nF -> 4.7uF; footprint Capacitor_SMD:C_0603_1608Metric -> Capacitor_SMD:C_1206_3216Metric
- J1: footprint Connector_PinHeader_2.00mm:PinHeader_1x08_P2.00mm_Vertical -> Connector_PinHeader_2.00mm:PinHeader_1x11_P2.00mm_Vertical; symbol Connector_Generic:Conn_01x08 -> Connector_Generic:Conn_01x11
Connections:
- net labels added: CANH, CANL, CANRX, CANTX, CURR_B, CURR_C, LEDG, LEDR, SH_B, SH_C
- wire segments 224 -> 290
Other:
- note added: "Thermal connection"
- moved on the sheet: C4, NT1, NTC1, R1, R12, R13

Commit message: Latest
Parts:
- removed NT2: Net-Tie_2, NetTie:NetTie-2_SMD_Pad0.5mm, symbol Device:Net-Tie_2
- removed R14: 0.001, Resistor_SMD:R_1210_3225Metric, symbol Device:R
- added R15: 0.001, Resistor_SMD:R_1210_3225Metric, symbol Device:R
- renumbered R15 to R14
Connections:
- net labels added: PHB_SH, PHC_SH
- net labels removed: SH_B, SH_C
- wire segments 290 -> 287
Other:
- moved on the sheet: R14
Changed lines of the file:
@@
 Wire Wire Line
 	9900 4250 9900 4300
-Wire Wire Line
-	9900 5950 9900 5900
 $Comp
 L power:+5V #PWR023
@@
 Wire Wire Line
 	5700 5150 5700 5200
-Wire Wire Line
-	5700 7250 5700 7100
 $Comp
 L power:+5V #PWR029
@@
 Text Label 10000 5300 0    50   ~ 0
 PH_B
-Wire Wire Line
-	9900 5300 10000 5300
 Text Label 5850 6200 0    50   ~ 0
 PH_C
-Wire Wire Line
-	5700 6200 5850 6200
 $Comp
 L power:GND #PWR020
@@
 L power:GNDPWR #PWR031
 U 1 1 5F03C982
-P 9900 6250
-F 0 "#PWR031" H 9900 6050 50  0001 C CNN
-F 1 "GNDPWR" H 9904 6096 50  0000 C CNN
-F 2 "" H 9900 6200 50  0001 C CNN
-F 3 "" H 9900 6200 50  0001 C CNN
-	1    9900 6250
+P 9900 5950
+F 0 "#PWR031" H 9900 5750 50  0001 C CNN
+F 1 "GNDPWR" H 9904 5796 50  0000 C CNN
+F 2 "" H 9900 5900 50  0001 C CNN
+F 3 "" H 9900 5900 50  0001 C CNN
+	1    9900 5950
 	1    0    0    -1
 $EndComp
@@
 L power:GNDPWR #PWR040
 U 1 1 5F06BFFF
-P 5700 7250
-F 0 "#PWR040" H 5700 7050 50  0001 C CNN
-F 1 "GNDPWR" H 5704 7096 50  0000 C CNN
-F 2 "" H 5700 7200 50  0001 C CNN
-F 3 "" H 5700 7200 50  0001 C CNN
-	1    5700 7250
+P 5700 6800
+F 0 "#PWR040" H 5700 6600 50  0001 C CNN
+F 1 "GNDPWR" H 5704 6646 50  0000 C CNN
+F 2 "" H 5700 6750 50  0001 C CNN
+F 3 "" H 5700 6750 50  0001 C CNN
+	1    5700 6800
 	1    0    0    -1
 $EndComp
@@
 Wire Wire Line
 	1650 5200 1450 5200
-$Comp
-L Device:R R14
-U 1 1 5FAA724B
-P 5700 6950
-F 0 "R14" H 5770 6996 50  0000 L CNN
-F 1 "0.001" H 5770 6905 50  0000 L CNN
-F 2 "Resistor_SMD:R_1210_3225Metric" V 5630 6950 50  0001 C CNN
-F 3 "~" H 5700 6950 50  0001 C CNN
-	1    5700 6950
-	1    0    0    -1
-$EndComp
-Wire Wire Line
-	5700 6800 5700 6750
-Wire Wire Line
-	5700 6750 5800 6750
-Connection ~ 5700 6750
-Wire Wire Line
-	5700 6750 5700 6700
-Text Label 5800 6750 0    50   ~ 0
-SH_C
-Text Label 6650 1800 2    50   ~ 0
-SH_C
-Wire Wire Line
-	6650 1800 6700 1800
-Wire Wire Line
-	6700 1550 6700 1800
 Text Notes 6200 1900 0    50   ~ 0
 Thermal connection
-$Comp
-L Device:R R15
-U 1 1 5FB13AA3
-P 9900 6100
-F 0 "R15" H 9970 6146 50  0000 L CNN
-F 1 "0.001" H 9970 6055 50  0000 L CNN
-F 2 "Resistor_SMD:R_1210_3225Metric" V 9830 6100 50  0001 C CNN
-F 3 "~" H 9900 6100 50  0001 C CNN
-	1    9900 6100
-	1    0    0    -1
-$EndComp
-Wire Wire Line
-	9900 5900 10000 5900
-Text Label 10000 5900 0    50   ~ 0
-SH_B
-Connection ~ 9900 5900
-Wire Wire Line
-	9900 5900 9900 5800
 $Comp
 L Amplifier_Current:NCS210 U8
@@
 	1    0    0    -1
 $EndComp
-Text Label 4400 1150 0    50   ~ 0
-SH_C
 $Comp
 L power:+3.3V #PWR0113
@@
 	1    0    0    -1
 $EndComp
-Text Label 4450 2400 0    50   ~ 0
-SH_B
-$Comp
-L power:GNDPWR #PWR0115
-U 1 1 5FBC9893
-P 4400 2600
-F 0 "#PWR0115" H 4400 2400 50  0001 C CNN
-F 1 "GNDPWR" H 4404 2446 50  0000 C CNN
-F 2 "" H 4400 2550 50  0001 C CNN
-F 3 "" H 4400 2550 50  0001 C CNN
-	1    4400 2600
-	1    0    0    -1
-$EndComp
 $Comp
 L power:GND #PWR0116
@@
 	1    0    0    -1
 $EndComp
-Wire Wire Line
-	4450 2400 4700 2400
-Wire Wire Line
-	4400 1150 4700 1150
 Text Label 5750 2300 0    50   ~ 0
-CURR_B
+CURR_C
 Wire Wire Line
 	5750 2300 5600 2300
 Text Label 5700 1050 0    50   ~ 0
-CURR_C
+CURR_B
 Wire Wire Line
 	5700 1050 5600 1050
@@
 $EndComp
 $Comp
-L power:GNDPWR #PWR0111
-U 1 1 5FB54838
-P 4700 1350
-F 0 "#PWR0111" H 4700 1150 50  0001 C CNN
-F 1 "GNDPWR" H 4704 1196 50  0000 C CNN
-F 2 "" H 4700 1300 50  0001 C CNN
-F 3 "" H 4700 1300 50  0001 C CNN
-	1    4700 1350
-	1    0    0    -1
-$EndComp
-$Comp
 L Amplifier_Current:NCS210 U9
 U 1 1 5FBC987E
@@
 	1    0    0    -1
 $EndComp
-$Comp
-L Device:Net-Tie_2 NT2
-U 1 1 603FE925
-P 4600 2600
-F 0 "NT2" H 4600 2689 50  0000 C CNN
-F 1 "Net-Tie_2" H 4600 2690 50  0001 C CNN
-F 2 "NetTie:NetTie-2_SMD_Pad0.5mm" H 4600 2600 50  0001 C CNN
-F 3 "~" H 4600 2600 50  0001 C CNN
-	1    4600 2600
-	1    0    0    -1
-$EndComp
-Wire Wire Line
-	4500 2600 4400 2600
+Wire Wire Line
+	9900 5800 9900 5950
+Wire Wire Line
+	5700 6700 5700 6800
+$Comp
+L Device:R R14
+U 1 1 5FB13AA3
+P 10550 5300
+F 0 "R14" H 10620 5346 50  0000 L CNN
+F 1 "0.001" H 10620 5255 50  0000 L CNN
+F 2 "Resistor_SMD:R_1210_3225Metric" V 10480 5300 50  0001 C CNN
+F 3 "~" H 10550 5300 50  0001 C CNN
+	1    10550 5300
+	0    1    1    0
+$EndComp
+$Comp
+L power:GNDPWR #PWR0123
+U 1 1 5EF583A9
+P 6700 1650
+F 0 "#PWR0123" H 6700 1450 50  0001 C CNN
+F 1 "GNDPWR" H 6704 1496 50  0000 C CNN
+F 2 "" H 6700 1600 50  0001 C CNN
+F 3 "" H 6700 1600 50  0001 C CNN
+	1    6700 1650
+	1    0    0    -1
+$EndComp
+Wire Wire Line
+	6700 1650 6700 1550
+Wire Wire Line
+	9900 5300 10400 5300
+Wire Wire Line
+	10700 5300 10850 5300
+Text Label 10850 5300 0    50   ~ 0
+PHB_SH
+$Comp
+L Device:R R15
+U 1 1 5EFE1CCD
+P 6300 6200
+F 0 "R15" H 6370 6246 50  0000 L CNN
+F 1 "0.001" H 6370 6155 50  0000 L CNN
+F 2 "Resistor_SMD:R_1210_3225Metric" V 6230 6200 50  0001 C CNN
+F 3 "~" H 6300 6200 50  0001 C CNN
+	1    6300 6200
+	0    1    1    0
+$EndComp
+Wire Wire Line
+	6450 6200 6600 6200
+Text Label 6600 6200 0    50   ~ 0
+PHC_SH
+Wire Wire Line
+	5700 6200 6150 6200
+Text Label 4300 2400 0    50   ~ 0
+PH_C
+Wire Wire Line
+	4300 2400 4700 2400
+Text Label 4300 2600 0    50   ~ 0
+PHC_SH
+Wire Wire Line
+	4300 2600 4700 2600
+Text Label 4300 1150 0    50   ~ 0
+PH_B
+Wire Wire Line
+	4300 1150 4700 1150
+Text Label 4300 1350 0    50   ~ 0
+PHB_SH
+Wire Wire Line
+	4300 1350 4700 1350
 $EndSCHEMATC
