File: BLDC-driver.kicad_pcb (KiCad board)
At the start: 2 copper layers, 55.9 x 56 mm, 60 parts, among them J1 Conn_01x06, J2 Conn_01x06, Q1 FDMS86550, Q2 FDMS86550, Q3 FDMS86550, Q4 FDMS86550, Q5 FDMS86550, Q6 FDMS86550, U1 ADP3120A, U2 STM32F103C8Tx, U3 AS5600, U4 ADP3120A, U5 ADP3120A, U6 MP2359, U7 MIC5504-3.3YM5

Commit message: Latest
Parts:
- added C29: 100nF, Capacitor_SMD:C_0603_1608Metric, F.Cu at (178.7, 107.2)
- added C30: 100nF, Capacitor_SMD:C_0402_1005Metric, F.Cu at (215.2, 124.3)
- added D2: LED, LED_SMD:LED_0603_1608Metric, F.Cu at (190.2, 134.9)
- added D3: LED, LED_SMD:LED_0603_1608Metric, F.Cu at (190.2, 136.4)
- added D4: 30V, Diode_SMD:D_SOD-523, F.Cu at (202.7, 108.4)
- added D5: 30V, Diode_SMD:D_SOD-523, F.Cu at (195.0, 109.6)
- added D6: 30V, Diode_SMD:D_SOD-523, F.Cu at (186.9, 109.4)
- added NT2: Net-Tie_2, NetTie:NetTie-2_SMD_Pad0.5mm, B.Cu at (202.4, 118.8)
- added R14: 0.001, Resistor_SMD:R_1210_3225Metric, B.Cu at (184.3, 108.5)
- added R15: 0.001, Resistor_SMD:R_1210_3225Metric, B.Cu at (201.2, 115.7)
- added R16: 120R, Resistor_SMD:R_0603_1608Metric, F.Cu at (187.0, 141.0)
- added R17: 1k, Resistor_SMD:R_0603_1608Metric, F.Cu at (186.1, 135.0)
- added R18: 1k, Resistor_SMD:R_0603_1608Metric, F.Cu at (187.6, 135.0)
- added R19: 10k, Resistor_SMD:R_0603_1608Metric, F.Cu at (178.8, 109.7)
- added R20: 10k, Resistor_SMD:R_0603_1608Metric, F.Cu at (178.8, 111.2)
- added R21: 10k, Resistor_SMD:R_0402_1005Metric, F.Cu at (217.1, 126.2)
- added R22: 10k, Resistor_SMD:R_0402_1005Metric, F.Cu at (218.1, 126.2)
- added U8: NCS210, Package_TO_SOT_SMD:SOT-363_SC-70-6, F.Cu at (181.1, 106.8)
- added U9: NCS210, Package_TO_SOT_SMD:SOT-363_SC-70-6, F.Cu at (214.7, 126.3)
- C27: value 100nF -> 4.7uF; footprint Capacitor_SMD:C_0603_1608Metric -> Capacitor_SMD:C_1206_3216Metric
- J1: footprint Connector_PinHeader_2.00mm:PinHeader_1x08_P2.00mm_Vertical -> Connector_PinHeader_2.00mm:PinHeader_1x11_P2.00mm_Vertical
- U3: value AS5600 -> MAX3051; footprint Package_SO:SOIC-8_3.9x4.9mm_P1.27mm -> Package_TO_SOT_SMD:SOT-23-8; moved to F.Cu
- moved C27 44.2 mm to (213.2, 107.8)
- moved J1 10.0 mm to (206.1, 143.4)
- moved U3 8.06 mm to (187.3, 121.5)
- moved C9 5.98 mm to (184.0, 121.3), turned to 90 degrees
- moved C4 5.48 mm to (176.8, 122.9), turned to 90 degrees
- moved C23 5.01 mm to (215.4, 113.6)
- moved U6 4.90 mm to (215.4, 111.1)
- moved R7 4.75 mm to (212.6, 110.6)
- moved J2 3.98 mm to (173.7, 129.9)
- moved R11 3.43 mm to (175.9, 130.1)
- moved R2 2.84 mm to (182.4, 138.7)
- moved R3 2.84 mm to (182.4, 137.2)
- moved C28 2.83 mm to (188.7, 130.7)
- moved C5 2.83 mm to (179.8, 121.7)
- moved C6 2.83 mm to (187.8, 125.0)
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Connections:
- C27 pad 1: GND -> +24V
- C27 pad 2: +3V3 -> GND
- C9 pad 1: GND -> +3V3
- C9 pad 2: +3V3 -> GND
- J1 pad 3: /SWDIO -> +3V3
- J1 pad 4: /SWCLK -> /SWDIO
- J1 pad 5: /SDA -> /SWCLK
- J1 pad 6: /SCL -> /SDA
- J1 pad 7: /TXD -> /SCL
- J1 pad 8: /RXD -> /TXD
- NTC1 pad 2: GNDPWR -> /SH_C
- Q4 pad 1: GNDPWR -> /SH_B
- Q4 pad 2: GNDPWR -> /SH_B
- Q4 pad 3: GNDPWR -> /SH_B
- Q6 pad 1: GNDPWR -> /SH_C
- Q6 pad 2: GNDPWR -> /SH_C
- Q6 pad 3: GNDPWR -> /SH_C
- U2 pad 11: Net-(U2-Pad11) -> /CURR_C
- U2 pad 12: Net-(U2-Pad12) -> /CURR_B
- U2 pad 14: Net-(U2-Pad14) -> /LEDR
- U2 pad 15: Net-(U2-Pad15) -> /LEDG
- U2 pad 32: Net-(U2-Pad32) -> /CANRX
- U2 pad 33: Net-(U2-Pad33) -> /CANTX
- U3 pad 1: +3V3 -> /CANTX
- U3 pad 2: +3V3 -> GND
- U3 pad 3: Net-(U3-Pad3) -> +3V3
- U3 pad 4: GND -> /CANRX
- U3 pad 5: Net-(U3-Pad5) -> GND
- U3 pad 6: /SDA -> /CANL
- U3 pad 7: /SCL -> /CANH
- U3 pad 8: Net-(U3-Pad8) -> GND
Routing:
- net GNDPWR: track 79.9 -> 130.2 mm, vias 62 -> 86
- net /CURR_B: track 0.00 -> 42.5 mm, vias 0 -> 2
- net /SH_B: track 0.00 -> 37.4 mm, vias 0 -> 1
- net /CURR_C: track 0.00 -> 34.9 mm, vias 0 -> 2
- net /CANH: track 0.00 -> 32.6 mm, vias 0 -> 3
- net /SDA: track 59.3 -> 28.6 mm
- net /CANL: track 0.00 -> 29.6 mm, vias 0 -> 3
- net +3V3: track 106.5 -> 134.9 mm, vias 5 -> 8
- net /SCL: track 52.4 -> 28.5 mm
- net Net-(NT2-Pad2): track 0.00 -> 21.2 mm, vias 0 -> 1
- net GND: track 33.8 -> 50.2 mm, vias 22 -> 43
- net +5V: track 109.8 -> 123.6 mm
- net /CANRX: track 0.00 -> 9.47 mm, vias 0 -> 2
- net /SWCLK: track 23.1 -> 32.3 mm
- net /CANTX: track 0.00 -> 8.62 mm, vias 0 -> 2
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- added copper zone on B.Cu, net /SH_C
Other:
- board size 55.9 x 56 mm -> 52.2 x 52.2 mm
- board text added: "+3V3"
- board text added: "+Vs"
- board text added: "3V3"
- board text added: "CANH"
- board text added: "CANL"
- board text added: "MISO"
- board text added: "MOSI"
- board text added: "Max 24V"
- board text added: "SCK"
- board text removed: "+24V"

Commit message: Latest
Parts:
- removed NT2: Net-Tie_2, NetTie:NetTie-2_SMD_Pad0.5mm
- moved C29 44.7 mm to (220.5, 123.0)
- moved R19 43.6 mm to (219.1, 126.3), turned to 270 degrees
- moved R20 41.6 mm to (217.6, 126.3), turned to 270 degrees
- moved R22 41.5 mm to (179.6, 110.8)
- moved R21 41.5 mm to (178.6, 110.7)
- moved U8 40.5 mm to (218.3, 122.8), turned to 90 degrees
- moved U9 39.9 mm to (179.3, 107.9), turned to 90 degrees
- moved C30 37.2 mm to (180.5, 110.7), turned to 90 degrees
- moved R14 26.0 mm to (209.9, 104.1), turned to 180 degrees
- moved R15 21.3 mm to (182.7, 105.3)
- moved NTC1 1.27 mm to (184.1, 105.5)
Connections:
- NTC1 pad 2: /SH_C -> GNDPWR
- Q4 pad 1: /SH_B -> GNDPWR
- Q4 pad 2: /SH_B -> GNDPWR
- Q4 pad 3: /SH_B -> GNDPWR
- Q6 pad 1: /SH_C -> GNDPWR
- Q6 pad 2: /SH_C -> GNDPWR
- Q6 pad 3: /SH_C -> GNDPWR
- R14 pad 1: /SH_C -> /PHB_SH
- R14 pad 2: GNDPWR -> /PH_B
- R15 pad 1: /SH_B -> /PHC_SH
- R15 pad 2: GNDPWR -> /PH_C
- U2 pad 18: Net-(U2-Pad18) -> (no net)
- U2 pad 19: Net-(U2-Pad19) -> (no net)
- U2 pad 2: Net-(U2-Pad2) -> (no net)
- U2 pad 20: Net-(U2-Pad20) -> (no net)
- U2 pad 21: Net-(U2-Pad21) -> (no net)
- U2 pad 22: Net-(U2-Pad22) -> (no net)
- U2 pad 25: Net-(U2-Pad25) -> (no net)
- U2 pad 26: Net-(U2-Pad26) -> (no net)
- U2 pad 27: Net-(U2-Pad27) -> (no net)
- U2 pad 28: Net-(U2-Pad28) -> (no net)
- U2 pad 3: Net-(U2-Pad3) -> (no net)
- U2 pad 4: Net-(U2-Pad4) -> (no net)
- U2 pad 5: Net-(U2-Pad5) -> (no net)
- U2 pad 6: Net-(U2-Pad6) -> (no net)
- U7 pad 4: Net-(U7-Pad4) -> (no net)
- U8 pad 4: /SH_C -> /PH_B
- U8 pad 5: GNDPWR -> /PHB_SH
- U8 pad 6: /CURR_C -> /CURR_B
- U9 pad 4: /SH_B -> /PH_C
- U9 pad 5: Net-(NT2-Pad2) -> /PHC_SH
- U9 pad 6: /CURR_B -> /CURR_C
Routing:
- net /SH_B: track 37.4 -> 0.00 mm, vias 1 -> 0
- net /PH_B: track 8.67 -> 41.7 mm, vias 18 -> 3
- net GNDPWR: track 130.2 -> 100.6 mm, vias 86 -> 94
- net /PHB_SH: track 0.00 -> 24.9 mm, vias 0 -> 7
- net Net-(NT2-Pad2): track 21.2 -> 0.00 mm, vias 1 -> 0
- net +3V3: track 134.9 -> 148.7 mm, vias 8 -> 9
- net /PH_C: track 12.1 -> 24.2 mm, vias 18 -> 4
- net /PHC_SH: track 0.00 -> 6.59 mm, vias 0 -> 7
- net /SH_C: track 6.52 -> 0.00 mm, vias 2 -> 0
- net /CURR_B: track 42.5 -> 48.3 mm
- net GND: track 50.2 -> 55.4 mm
- net /CURR_C: track 34.9 -> 32.1 mm
- net Net-(R21-Pad1): track 2.57 -> 4.14 mm
- net /FET_TEMP: track 39.6 -> 38.6 mm
- net +5V: track 123.6 -> 122.7 mm
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- added copper zone on F.Cu, net /PHB_SH
- added copper zone on F.Cu, net /PHC_SH
- removed copper zone on F.Cu, net /PH_B
- removed copper zone on F.Cu, net /PH_C
- removed copper zone on B.Cu, net /SH_C

Commit message: Latest
Parts:
- added C31: 100nF, Capacitor_SMD:C_0402_1005Metric, F.Cu at (176.4, 114.4)
- added C32: 100nF, Capacitor_SMD:C_0402_1005Metric, F.Cu at (185.6, 137.0)
- added D7: D_TVS, Diode_SMD:D_SMB, F.Cu at (212.2, 129.6)
- added R23: 10k, Resistor_SMD:R_0402_1005Metric, F.Cu at (177.1, 112.5)
- added R24: 10k, Resistor_SMD:R_0402_1005Metric, F.Cu at (185.5, 138.0)
- D4, D5, D6: value 30V -> 45V
- moved NTC1 1.57 mm to (183.0, 106.6)
Connections:
- U2 pad 11: /CURR_C -> /CURR_C_FLT
- U2 pad 12: /CURR_B -> /CURR_B_FLT
- U2 pad 18: (no net) -> Net-(U2-Pad18)
- U2 pad 19: (no net) -> Net-(U2-Pad19)
- U2 pad 2: (no net) -> Net-(U2-Pad2)
- U2 pad 20: (no net) -> Net-(U2-Pad20)
- U2 pad 21: (no net) -> Net-(U2-Pad21)
- U2 pad 22: (no net) -> Net-(U2-Pad22)
- U2 pad 25: (no net) -> Net-(U2-Pad25)
- U2 pad 26: (no net) -> Net-(U2-Pad26)
- U2 pad 27: (no net) -> Net-(U2-Pad27)
- U2 pad 28: (no net) -> Net-(U2-Pad28)
- U2 pad 3: (no net) -> Net-(U2-Pad3)
- U2 pad 4: (no net) -> Net-(U2-Pad4)
- U2 pad 5: (no net) -> Net-(U2-Pad5)
- U2 pad 6: (no net) -> Net-(U2-Pad6)
- U7 pad 4: (no net) -> Net-(U7-Pad4)
Routing:
- net /CURR_C_FLT: track 0.00 -> 27.0 mm, vias 0 -> 2
- net /CURR_C: track 32.1 -> 5.68 mm, vias 2 -> 0
- net /CURR_B_FLT: track 0.00 -> 6.73 mm
- net /CURR_B: track 48.3 -> 41.7 mm
- net /FET_TEMP: track 38.6 -> 36.0 mm
- net GNDPWR: track 100.6 -> 102.9 mm, vias 94 -> 97
- net /PWM_B: track 72.8 -> 74.1 mm, vias 4 -> 5
- net +5V: track 122.7 -> 123.4 mm
- net /PH_B: track 41.7 -> 42.2 mm
- net /PWM_C: track 22.4 -> 22.9 mm
- net +24V: track 88.0 -> 88.2 mm, vias 62 -> 70
- net GND: vias 43 -> 64
